Commit message: added 4 sensors in the urdf&code

File: AdvanDiptera_discription/urdf/AdvanDiptera.xacro (robot description, xacro)
@@ -28,21 +28,21 @@
     <xacro:sonar_sensor name="sonarD" parent="base_link" ros_topic="/sonar_Tp0
 " update_rate="10" min_range="0.03" max_range="3.0" field_of_view="${40*pi/180}" ray_count="3">
-      <origin xyz="-0.01 0.0 0.09" rpy="0 ${90*pi/180} 0"/>
+      <origin xyz="-0.05 -0.01 0.09" rpy="0 ${90*pi/180} 0"/>
     </xacro:sonar_sensor>
   <xacro:sonar_sensor name="sonarF" parent="base_link" ros_topic="/sonar_Tp1
 " update_rate="10" min_range="0.03" max_range="3.0" field_of_view="${40*pi/180}" ray_count="3">
-      <origin xyz="-0.01 0.02 0.09" rpy="0 ${pi/180} 0"/>
+      <origin xyz="-0.3 0.0 0.09" rpy="0 ${pi/180} ${pi}"/>
     </xacro:sonar_sensor>
   <xacro:sonar_sensor name="sonarL" parent="base_link" ros_topic="/sonar_Tp2
 " update_rate="10" min_range="0.03" max_range="3.0" field_of_view="${40*pi/180}" ray_count="3">
-      <origin xyz="-0.01 -0.02 0.09" rpy="0 ${pi/180} 90"/>
+      <origin xyz="-0.06 -0.3 0.09" rpy="0 ${pi/180} ${270*pi/180}"/>
     </xacro:sonar_sensor>
   <xacro:sonar_sensor name="sonarR" parent="base_link" ros_topic="/sonar_Tp3
 " update_rate="10" min_range="0.03" max_range="3.0" field_of_view="${40*pi/180}" ray_count="3">
-      <origin xyz="-0.02 0.02 0.09" rpy="0 ${pi/180} 180"/>
+      <origin xyz="-0.06 0.3 0.09" rpy="0 ${pi/180} ${90*pi/180}"/>
     </xacro:sonar_sensor>
   <xacro:sonar_sensor name="sonarB" parent="base_link" ros_topic="/sonar_Tp4
 " update_rate="10" min_range="0.03" max_range="3.0" field_of_view="${40*pi/180}" ray_count="3">
-      <origin xyz="0.02 0.02 0.09" rpy="0 ${pi/180} 270"/>
+      <origin xyz="0.2 0.0 0.09" rpy="0 ${pi/180} ${pi/180}"/>
     </xacro:sonar_sensor>
 </robot>
